File: arduino_box/Arduino.sch (KiCad schematic (older format))
At the start: 31 parts, among them K1 K, K2 K, P1 5.5x2.1, P10 CON3, P11 CE, P12 C13, P13 3.5mm, P14 MTE-3, P2 5.5x2.1, P3 5.5x2.1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

Commit message: kicad schematics
Other:
- note added: "Band"
- note added: "DL9LJ - November 2016"
- note removed: "Remote"
Changed lines of the file:
@@
 Wire Wire Line
 	4450 2400 6400 2400
-Text Notes 7400 2550 0    60   ~ 0
-Remote
 Wire Wire Line
 	5100 6000 5100 5950
@@
 Text Notes 600  3900 0    60   ~ 0
 12V
+Text Notes 7400 2550 0    60   ~ 0
+Band
+Text Notes 5000 11050 0    60   ~ 0
+DL9LJ - November 2016
 $EndSCHEMATC
